File: mux2Schematic/mux2Schematic.kicad_sch (KiCad schematic)
At the start: 64 parts, among them J1 Conn_02x12_Odd_Even, J10 Conn_02x06_Top_Bottom, J11 Conn_02x06_Top_Bottom, J12 Conn_02x06_Top_Bottom, J13 Conn_02x06_Top_Bottom, J14 Conn_02x06_Top_Bottom, J15 Conn_01x02, J16 Conn_01x02, J17 Conn_01x02, J18 Conn_01x02, J19 Conn_01x02, J2 Conn_02x06_Top_Bottom, J20 Conn_01x02, J21 Conn_01x02, J3 Banana, J30 Conn_01x8, J31 Conn_01x8, J32 Conn_01x02, J33 Conn_01x02, J34 Conn_01x02, J35 Conn_01x02, J36 Conn_01x02, J37 Conn_01x02, J38 Conn_01x02, J39 Conn_01x02, J4 Banana, J5 Conn_01x8, J6 Conn_01x02, J7 Conn_02x06_Top_Bottom, J8 Conn_01x10, J9 Conn_02x06_Top_Bottom, U1 CD74HC4051E, U2 AMS1117-1.8, U3 AZ1084-3.3

Commit message: PCB finished!
Haven't thoroughly looked it over yet
Parts:
- added D1, D10, D11, D12, D13, D14, D15, D16, D17, D18, D19, D20, D21, D22, D23, D24, D7, D8, D9: HSMA-C170, LED_SMD:LED_0805_2012Metric, symbol Device:LED
- added JP1: SolderJumper_2_Bridged, Jumper:SolderJumper-2_P1.3mm_Bridged_RoundedPad1.0x1.5mm, symbol Jumper:SolderJumper_2_Bridged
- added R10, R11, R12, R14, R15, R16, R17, R18, R19, R20, R21, R22, R23, R24, R25, R26, R27, R9: 2.2k, Resistor_SMD:R_0805_2012Metric, symbol Device:R
- added R13: 5.1k, Resistor_SMD:R_0805_2012Metric, symbol Device:R
- C1: symbol Device:C -> Device:C_Small
- C2, C3, C4, C5: symbol Device:C_Polarized -> Device:C_Small
- R1, R2, R3, R4, R5, R6, R7, R8: value 10k -> 5.1k
- renumbered JP3 to JP2
Connections:
- net CIPO: now also J1.10 (Pin_10), J8.7 (Pin_7), D1.2 (A); no longer J1.16 (Pin_16)
- net COPI: now also D16.2 (A)
- net CS: now also J8.4 (Pin_4), D12.2 (A); no longer J8.6 (Pin_6)
- net CS_0: now also U1.15 (A2), D13.2 (A); no longer U1.13 (A0)
- net CS_1: now also D17.2 (A)
- net CS_2: now also U1.13 (A0), D18.2 (A); no longer U1.15 (A2)
- net CS_3: now also D19.2 (A)
- net CS_4: now also D21.2 (A)
- net CS_5: now also U1.2 (A6), D22.2 (A); no longer U1.5 (A5)
- net CS_6: now also U1.4 (A7), D23.2 (A); no longer U1.2 (A6)
- net CS_7: now also U1.5 (A5), D24.2 (A); no longer U1.4 (A7)
- net GND: now also D15.1 (K), JP1.1 (A); no longer J8.10 (Pin_10)
- net S0: now also D7.2 (A)
- net S1: now also D8.2 (A)
- net S2: now also D9.2 (A)
- net SCLK: now also J1.16 (Pin_16), J8.6 (Pin_6), D10.2 (A); no longer J1.12 (Pin_12), J8.4 (Pin_4)
- net VCC: now also R13.2
- net ~{CLR}: now also J8.10 (Pin_10), D14.2 (A); no longer J8.9 (Pin_9)
- net ~{LDAC}: now also J1.6 (Pin_6), J8.8 (Pin_8), D11.2 (A); no longer J1.10 (Pin_10), J8.7 (Pin_7)
- net ~{RESET}: now also J1.12 (Pin_12), J8.9 (Pin_9), D20.2 (A); no longer J1.6 (Pin_6), J8.8 (Pin_8)
- new net: JP1.2 (B), R10.1, R11.1, R12.1, R14.1, R15.1, R16.1, R17.1, R18.1, R19.1, R20.1, R21.1, R22.1, R23.1, R24.1, R25.2, R26.2, R27.1, R9.1
- new net: D7.1 (K), R15.2
- new net: D15.2 (A), R13.1
- new net: D10.1 (K), R18.2
- new net: D20.1 (K), R22.2
- new net: D23.1 (K), R25.1
- new net: D18.1 (K), R20.2
- new net: D9.1 (K), R17.2
- new net: D22.1 (K), R24.2
- new net: D16.1 (K), R14.2
- new net: D12.1 (K), R11.2
- new net: D13.1 (K), R12.2
- new net: D1.1 (K), R27.2
- new net: D11.1 (K), R10.2
- new net: D14.1 (K), R9.2
- new net: D24.1 (K), R26.1
- new net: D17.1 (K), R19.2
- new net: D8.1 (K), R16.2
- new net: D21.1 (K), R23.2
- new net: D19.1 (K), R21.2
Other:
- note added: "LED indicators"
- moved on the sheet: C1, H1, H2, H3, H4, H5, H6, H7, H8, J1, J15, J16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

Commit message: nvm it's not done
fixed most of the problem
Parts:
- added J40: Conn_01x06, symbol Connector_Generic:Conn_01x06
- J10: renamed from J13; value Conn_02x06_Top_Bottom -> Conn_02x06_Odd_Even; symbol Connector_Generic:Conn_02x06_Top_Bottom -> Connector_Generic:Conn_02x06_Odd_Even
- J13: renamed from J11; value Conn_02x06_Top_Bottom -> Conn_02x06_Odd_Even; symbol Connector_Generic:Conn_02x06_Top_Bottom -> Connector_Generic:Conn_02x06_Odd_Even
- J15: renamed from J10; value Conn_02x06_Top_Bottom -> Conn_02x06_Odd_Even; symbol Connector_Generic:Conn_02x06_Top_Bottom -> Connector_Generic:Conn_02x06_Odd_Even
- J17: renamed from J9; value Conn_02x06_Top_Bottom -> Conn_02x06_Odd_Even; symbol Connector_Generic:Conn_02x06_Top_Bottom -> Connector_Generic:Conn_02x06_Odd_Even
- J18: renamed from J7; value Conn_02x06_Top_Bottom -> Conn_02x06_Odd_Even; symbol Connector_Generic:Conn_02x06_Top_Bottom -> Connector_Generic:Conn_02x06_Odd_Even
- J21: renamed from J2; value Conn_02x06_Top_Bottom -> Conn_02x06_Odd_Even; symbol Connector_Generic:Conn_02x06_Top_Bottom -> Connector_Generic:Conn_02x06_Odd_Even
- J7: renamed from J14; value Conn_02x06_Top_Bottom -> Conn_02x06_Odd_Even; symbol Connector_Generic:Conn_02x06_Top_Bottom -> Connector_Generic:Conn_02x06_Odd_Even
- J8: renamed from J12; value Conn_02x06_Top_Bottom -> Conn_02x06_Odd_Even; symbol Connector_Generic:Conn_02x06_Top_Bottom -> Connector_Generic:Conn_02x06_Odd_Even
- renumbered C3 to C1, C4 to C3, C5 to C4, C1 to C5, D15 to D1, D11 to D10, D1 to D11, D10 to D13, D9 to D14, D16 to D15, D8 to D16, D7 to D17, D14 to D18, D20 to D19, D24 to D2, D22 to D3, D23 to D4, D17 to D5, D13 to D6, D21 to D7, D19 to D8, D18 to D9, H2 to H1, H4 to H2, H1 to H3, H3 to H4, J34 to J11, J35 to J12, J36 to J14, J37 to J16, J38 to J19, J3 to J2, J39 to J20, J6 to J22, J22 to J23, J15 to J24, J5 to J25, J23 to J26, J16 to J27, J24 to J28, J25 to J29, J4 to J3, J17 to J30, J26 to J31, J18 to J32, J27 to J33, J19 to J34, J31 to J35, J20 to J36, J28 to J37, J29 to J38, J21 to J39, J30 to J4, J8 to J5, J32 to J6, J33 to J9, JP2 to JP1, JP1 to JP2, R13 to R1, R25 to R10, R21 to R11, R23 to R13, R24 to R14, R26 to R15, R20 to R16, R19 to R17, R15 to R18, R27 to R19, R7 to R2, R14 to R20, R16 to R21, R18 to R22, R11 to R23, R10 to R24, R17 to R25, R22 to R26, R9 to R27, R2 to R3, R3 to R5, R1 to R6, R5 to R7, R6 to R8, R8 to R9, U3 to U1, U1 to U3
Connections:
- net CIPO: now also J1.16 (Pin_16), J10.7 (Pin_7), J13.7 (Pin_7), J15.7 (Pin_7), J17.7 (Pin_7), J18.7 (Pin_7), J21.7 (Pin_7), J7.7 (Pin_7), J8.7 (Pin_7); no longer J1.10 (Pin_10), J10.3 (Pin_3), J13.3 (Pin_3), J15.3 (Pin_3), J17.3 (Pin_3), J18.3 (Pin_3), J21.3 (Pin_3), J7.3 (Pin_3), J8.3 (Pin_3)
- net COPI: now also J1.12 (Pin_12), J10.9 (Pin_9), J13.9 (Pin_9), J15.9 (Pin_9), J17.9 (Pin_9), J18.9 (Pin_9), J21.9 (Pin_9), J7.9 (Pin_9), J8.9 (Pin_9); no longer J1.18 (Pin_18), J10.2 (Pin_2), J13.2 (Pin_2), J15.2 (Pin_2), J17.2 (Pin_2), J18.2 (Pin_2), J21.2 (Pin_2), J7.2 (Pin_2), J8.2 (Pin_2)
- net CS_0: now also J21.11 (Pin_11); no longer J21.1 (Pin_1)
- net CS_1: now also J18.11 (Pin_11); no longer J18.1 (Pin_1)
- net CS_2: now also J17.11 (Pin_11); no longer J17.1 (Pin_1)
- net CS_3: now also J15.11 (Pin_11); no longer J15.1 (Pin_1)
- net CS_4: now also J13.11 (Pin_11); no longer J13.1 (Pin_1)
- net CS_5: now also J10.11 (Pin_11); no longer J10.1 (Pin_1)
- net CS_6: now also J8.11 (Pin_11); no longer J8.1 (Pin_1)
- net CS_7: now also J7.11 (Pin_11); no longer J7.1 (Pin_1)
- net GND: now also J10.3 (Pin_3), J10.4 (Pin_4), J13.3 (Pin_3), J13.4 (Pin_4), J15.3 (Pin_3), J15.4 (Pin_4), J17.3 (Pin_3), J17.4 (Pin_4), J18.3 (Pin_3), J18.4 (Pin_4), J21.3 (Pin_3), J21.4 (Pin_4), J7.3 (Pin_3), J7.4 (Pin_4), J8.3 (Pin_3), J8.4 (Pin_4); no longer J10.11 (Pin_11), J10.5 (Pin_5), J13.11 (Pin_11), J13.5 (Pin_5), J15.11 (Pin_11), J15.5 (Pin_5), J17.11 (Pin_11), J17.5 (Pin_5), J18.11 (Pin_11), J18.5 (Pin_5), J21.11 (Pin_11), J21.5 (Pin_5), J7.11 (Pin_11), J7.5 (Pin_5), J8.11 (Pin_11), J8.5 (Pin_5)
- net IOVcc: now also J10.1 (Pin_1), J10.2 (Pin_2), J13.1 (Pin_1), J13.2 (Pin_2), J15.1 (Pin_1), J15.2 (Pin_2), J17.1 (Pin_1), J17.2 (Pin_2), J18.1 (Pin_1), J18.2 (Pin_2), J21.1 (Pin_1), J21.2 (Pin_2), J7.1 (Pin_1), J7.2 (Pin_2), J8.1 (Pin_1), J8.2 (Pin_2); no longer J10.12 (Pin_12), J10.6 (Pin_6), J13.12 (Pin_12), J13.6 (Pin_6), J15.12 (Pin_12), J15.6 (Pin_6), J17.12 (Pin_12), J17.6 (Pin_6), J18.12 (Pin_12), J18.6 (Pin_6), J21.12 (Pin_12), J21.6 (Pin_6), J7.12 (Pin_12), J7.6 (Pin_6), J8.12 (Pin_12), J8.6 (Pin_6)
- net SCLK: now also J1.18 (Pin_18), J10.5 (Pin_5), J13.5 (Pin_5), J15.5 (Pin_5), J17.5 (Pin_5), J18.5 (Pin_5), J21.5 (Pin_5), J7.5 (Pin_5), J8.5 (Pin_5); no longer J1.16 (Pin_16), J10.4 (Pin_4), J13.4 (Pin_4), J15.4 (Pin_4), J17.4 (Pin_4), J18.4 (Pin_4), J21.4 (Pin_4), J7.4 (Pin_4), J8.4 (Pin_4)
- net VCC: now also J40.2 (Pin_2)
- net ~{CLR}: now also J1.10 (Pin_10), J10.8 (Pin_8), J13.8 (Pin_8), J15.8 (Pin_8), J17.8 (Pin_8), J18.8 (Pin_8), J21.8 (Pin_8), J7.8 (Pin_8), J8.8 (Pin_8); no longer J1.4 (Pin_4), J10.9 (Pin_9), J13.9 (Pin_9), J15.9 (Pin_9), J17.9 (Pin_9), J18.9 (Pin_9), J21.9 (Pin_9), J7.9 (Pin_9), J8.9 (Pin_9)
- net ~{LDAC}: now also J1.4 (Pin_4), J10.12 (Pin_12), J13.12 (Pin_12), J15.12 (Pin_12), J17.12 (Pin_12), J18.12 (Pin_12), J21.12 (Pin_12), J7.12 (Pin_12), J8.12 (Pin_12); no longer J1.6 (Pin_6), J10.7 (Pin_7), J13.7 (Pin_7), J15.7 (Pin_7), J17.7 (Pin_7), J18.7 (Pin_7), J21.7 (Pin_7), J7.7 (Pin_7), J8.7 (Pin_7)
- net ~{RESET}: now also J1.6 (Pin_6), J10.10 (Pin_10), J13.10 (Pin_10), J15.10 (Pin_10), J17.10 (Pin_10), J18.10 (Pin_10), J21.10 (Pin_10), J7.10 (Pin_10), J8.10 (Pin_10); no longer J1.12 (Pin_12), J10.8 (Pin_8), J13.8 (Pin_8), J15.8 (Pin_8), J17.8 (Pin_8), J18.8 (Pin_8), J21.8 (Pin_8), J7.8 (Pin_8), J8.8 (Pin_8)
- no-connect marks 14 -> 19
Other:
- note added: "1"
- note added: "VCC IDC Connector"
