File: mux2Schematic/mux2Schematic.kicad_sch (KiCad schematic)
At the start: 104 parts, among them J1 Conn_02x12_Odd_Even, J10 Conn_02x06_Odd_Even, J11 Conn_01x02, J12 Conn_01x02, J13 Conn_02x06_Odd_Even, J14 Conn_01x02, J15 Conn_02x06_Odd_Even, J16 Conn_01x02, J17 Conn_02x06_Odd_Even, J18 Conn_02x06_Odd_Even, J19 Conn_01x02, J2 Banana, J20 Conn_01x02, J21 Conn_02x06_Odd_Even, J22 Conn_01x02, J24 Conn_01x02, J25 Conn_01x8, J27 Conn_01x02, J3 Banana, J30 Conn_01x02, J32 Conn_01x02, J34 Conn_01x02, J35 Conn_01x8, J36 Conn_01x02, J39 Conn_01x02, J4 Conn_01x8, J40 Conn_01x06, J5 Conn_01x10, J6 Conn_01x02, J7 Conn_02x06_Odd_Even, J8 Conn_02x06_Odd_Even, J9 Conn_01x02, U1 AZ1084-3.3, U2 AMS1117-1.8, U3 CD74HC4051E

Commit message: PCB Finalized & Ordered!
Had to manually fix a number of things (e.g. component rotation) when I ordered it on JLCPCB. I didn't add the settings that let you rotate the part automatically into the right position.
Parts:
- D1, D10, D11, D12, D13, D14, D15, D16, D17, D18, D19, D2, D3, D4, D5, D6, D7, D8, D9: JLCPCB Part # (none) -> C7466711
- J1: JLCPCB Part # (none) -> C132440
- J10, J13, J15, J17, J18, J21, J7, J8: JLCPCB Part # (none) -> C2897426
- J11, J12, J14, J16, J19, J20, J22, J24, J27, J30, J32, J34, J36, J39, J6, J9: JLCPCB Part # (none) -> C49661
- J2: JLCPCB Part # (none) -> C106273
- J23, J26, J28, J29, J31, J33, J37, J38: JLCPCB Part # (none) -> C496549
- J25, J35, J4: JLCPCB Part # (none) -> C2829996
- J3: JLCPCB Part # (none) -> C106272
- J40: now left out of the parts list
- J5: JLCPCB Part # (none) -> C5156617
- R1: value 5.1k -> 2.2k
- R2, R3, R4, R5, R6, R7, R8, R9: value 5.1k -> 10k
- U1: value AZ1084-3.3 -> AZ1084CD-3.3TRG1; JLCPCB Part # (none) -> C151391
- U2: JLCPCB Part # (none) -> C347220
- U3: value CD74HC4051E -> CD74HC4053PWR; JLCPCB Part # (none) -> C6546
Connections:
- net CIPO: now also J5.9 (Pin_9); no longer J5.7 (Pin_7)
- net COPI: now also J5.10 (Pin_10); no longer J5.5 (Pin_5)
- net GND: now also J40.1 (Pin_1)
- net SCLK: now also J5.8 (Pin_8); no longer J5.6 (Pin_6)
- net ~{CLR}: now also J5.7 (Pin_7); no longer J5.10 (Pin_10)
- net ~{LDAC}: now also J5.5 (Pin_5); no longer J5.8 (Pin_8)
- net ~{RESET}: now also J5.6 (Pin_6); no longer J5.9 (Pin_9)
- no-connect marks 19 -> 18
Other:
- moved on the sheet: J1
